Commit message: done testing 2 DOF

File: models/others/robots/2DOF_description/urdf/2DOF_description.urdf (robot description, URDF)
Before this commit: robot parallelepiped, 3 links, 2 joints
Links:
- added link world
Joints:
- added joint world_joint: type fixed, parent world, child base_link, origin xyz=0.0 0.0 0.0 rpy=0.0 0.0 0.0
- joint joint1: origin xyz=0.25 0 0.25 rpy=0 -0.785398 0 -> xyz=0.25 0 0.25 rpy=0 0 0

Commit message: add identificationwith external wrench

File: models/others/robots/2DOF_description/urdf/2DOF_description.urdf (robot description, URDF)
Before this commit: robot parallelepiped, 4 links, 3 joints
Links:
- removed link world
Joints:
- removed joint world_joint

File: models/others/robots/SC_3DOF/urdf/3DOF.urdf (robot description, URDF)
Before this commit: robot Chaser, 6 links, 5 joints
Joints:
- joint Joint_1: limit (none) -> lower=0 upper=0 effort=0 velocity=0
- joint Joint_2: limit (none) -> lower=0 upper=0 effort=0 velocity=0
- joint Joint_3: limit (none) -> lower=0 upper=0 effort=0 velocity=0
